File: coincounter/coincounter/flashtool.kicad_sch (KiCad schematic)
At the start: 50 parts

Commit message: Desktop work
Parts:
- removed R?: 100K, symbol Device:R
- added R? (x2): 100K, symbol Device:R
- R?: value 100K -> 20K
Connections:
- net GND: now also R?.1, R?.1; no longer U?.19 (AVref)
- net at U?.18 (P110/AN0): now also R?.2
- new net: R?.2, U?.19 (AVref)
