File: coincounter/schematics/flashtool.kicad_sch (KiCad schematic)
At the start: 51 parts

Commit message: Reorganize all the things, add some extra sanity checking and bring everything up to date with reality. Additionally add a README describing everything in coincounter.
Parts:
- removed J?: Conn_01x08, symbol Connector_Generic:Conn_01x08
- removed R?: 100K, symbol Device:R
- added J?: Conn_01x01, symbol Connector_Generic:Conn_01x01
- added J?: Conn_01x07, symbol Connector_Generic:Conn_01x07
- added J?: Conn_01x03, symbol Connector_Generic:Conn_01x03
- added R?: 20K, symbol Device:R
- R?: value 20K -> 100K
Connections:
- net GND: now also J?.2 (Pin_2), J?.7 (Pin_7); no longer R?.2, R?.2, R?.2, R?.2, R?.2, R?.2, R?.2, R?.2
- net at C?.2, U?.20 (Vpp): now also J?.3 (Pin_3)
- net at C?.2, U?.21 (Vdd): now also J?.1 (Pin_1)
- net at R?.1: now also J?.4 (Pin_4)
- net at U?.3 (~{RESET}): now also R?.2
- net at R?.1: now also J?.3 (Pin_3)
- net at R?.1: now also J?.2 (Pin_2)
- net at R?.1: now also J?.5 (Pin_5)
- net at R?.1: now also J?.6 (Pin_6)
- new net: J?.1 (Pin_1), R?.2, R?.2, R?.2, R?.2, R?.2, R?.2, R?.2, R?.2
- new net: J?.1 (Pin_1), R?.1
Other:
- moved on the sheet: J?
