File: ledmatrix/comms.kicad_sch (KiCad schematic)
At the start: 7 parts

Commit message: Temp commit to move computers.
Parts:
- added J?: Conn_02x03_Top_Bottom, symbol Connector_Generic:Conn_02x03_Top_Bottom
Connections:
- net GND: now also J?.4 (Pin_4), J?.5 (Pin_5), J?.6 (Pin_6)
- net VCC: now also J?.1 (Pin_1), J?.2 (Pin_2), J?.3 (Pin_3)
Other:
- moved on the sheet: J?, R?, U?
