File: ledmatrix/scanlines.kicad_sch (KiCad schematic)
At the start: 101 parts

Commit message: Temp commit to move computers.
Connections:
- new net: U?.14 (Q0), U?.2 (A0), U?.2 (A0)
- new net: U?.12 (Q2), U?.21 (A2), U?.21 (A2)
- new net: U?.11 (Q3), U?.22 (A3), U?.22 (A3)
- new net: U?.13 (Q1), U?.3 (A1), U?.3 (A1)
Changed lines of the file:
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@@
 (kicad_sch (version 20211123) (generator eeschema)
   (paper "A3")
-  (junction (at 302.26 46.99) (diameter 0) (color 0 0 0 0)
-  )
   (junction (at 233.68 59.69) (diameter 0) (color 0 0 0 0)
   )
@@
   (junction (at 238.76 170.18) (diameter 0) (color 0 0 0 0)
   )
-  (junction (at 300.99 44.45) (diameter 0) (color 0 0 0 0)
-  )
   (junction (at 292.1 90.17) (diameter 0) (color 0 0 0 0)
   )
@@
   )
   (junction (at 215.9 274.32) (diameter 0) (color 0 0 0 0)
-  )
-  (junction (at 303.53 49.53) (diameter 0) (color 0 0 0 0)
   )
   (junction (at 243.84 149.86) (diameter 0) (color 0 0 0 0)
@@
     (stroke (width 0) (type default) (color 0 0 0 0))
   )
-  (wire (pts (xy 303.53 49.53) (xy 303.53 46.99))
-    (stroke (width 0) (type default) (color 0 0 0 0))
-  )
   (wire (pts (xy 345.44 35.56) (xy 345.44 41.91))
     (stroke (width 0) (type default) (color 0 0 0 0))
@@
     (stroke (width 0) (type default) (color 0 0 0 0))
   )
-  (wire (pts (xy 302.26 46.99) (xy 302.26 104.14))
+  (wire (pts (xy 302.26 44.45) (xy 302.26 104.14))
     (stroke (width 0) (type default) (color 0 0 0 0))
   )
@@
     (stroke (width 0) (type default) (color 0 0 0 0))
   )
-  (wire (pts (xy 281.94 44.45) (xy 300.99 44.45))
-    (stroke (width 0) (type default) (color 0 0 0 0))
-  )
   (wire (pts (xy 252.73 160.02) (xy 241.3 160.02))
     (stroke (width 0) (type default) (color 0 0 0 0))
@@
     (stroke (width 0) (type default) (color 0 0 0 0))
   )
-  (wire (pts (xy 300.99 44.45) (xy 300.99 41.91))
+  (wire (pts (xy 300.99 41.91) (xy 300.99 101.6))
     (stroke (width 0) (type default) (color 0 0 0 0))
   )
@@
     (stroke (width 0) (type default) (color 0 0 0 0))
   )
-  (wire (pts (xy 303.53 49.53) (xy 304.8 49.53))
-    (stroke (width 0) (type default) (color 0 0 0 0))
-  )
   (wire (pts (xy 146.05 59.69) (xy 147.32 59.69))
     (stroke (width 0) (type default) (color 0 0 0 0))
@@
     (stroke (width 0) (type default) (color 0 0 0 0))
   )
-  (wire (pts (xy 300.99 44.45) (xy 302.26 44.45))
+  (wire (pts (xy 281.94 44.45) (xy 302.26 44.45))
     (stroke (width 0) (type default) (color 0 0 0 0))
   )
@@
     (stroke (width 0) (type default) (color 0 0 0 0))
   )
-  (wire (pts (xy 303.53 106.68) (xy 303.53 49.53))
+  (wire (pts (xy 303.53 46.99) (xy 303.53 106.68))
     (stroke (width 0) (type default) (color 0 0 0 0))
   )
@@
     (stroke (width 0) (type default) (color 0 0 0 0))
   )
-  (wire (pts (xy 281.94 49.53) (xy 303.53 49.53))
+  (wire (pts (xy 281.94 49.53) (xy 304.8 49.53))
     (stroke (width 0) (type default) (color 0 0 0 0))
   )
@@
     (stroke (width 0) (type default) (color 0 0 0 0))
   )
-  (wire (pts (xy 281.94 46.99) (xy 302.26 46.99))
+  (wire (pts (xy 281.94 46.99) (xy 303.53 46.99))
     (stroke (width 0) (type default) (color 0 0 0 0))
   )
@@
     (stroke (width 0) (type default) (color 0 0 0 0))
   )
-  (wire (pts (xy 302.26 44.45) (xy 302.26 46.99))
-    (stroke (width 0) (type default) (color 0 0 0 0))
-  )
   (wire (pts (xy 246.38 46.99) (xy 246.38 49.53))
     (stroke (width 0) (type default) (color 0 0 0 0))
@@
     (stroke (width 0) (type default) (color 0 0 0 0))
   )
-  (wire (pts (xy 300.99 101.6) (xy 300.99 44.45))
-    (stroke (width 0) (type default) (color 0 0 0 0))
-  )
   (wire (pts (xy 383.54 30.48) (xy 383.54 43.18))
     (stroke (width 0) (type default) (color 0 0 0 0))
@@
     (stroke (width 0) (type default) (color 0 0 0 0))
   )
-  (wire (pts (xy 302.26 46.99) (xy 303.53 46.99))
-    (stroke (width 0) (type default) (color 0 0 0 0))
-  )
