File: ledmatrix/LEDdriver.kicad_sch (KiCad schematic)
At the start: 2 parts

Commit message: Temp commit to move computers.
Connections:
- net SOUT: now reaches U?.5 (SOUT)
- no-connect marks 1 -> 0
Changed lines of the file:
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@@
   (junction (at 101.6 140.97) (diameter 0) (color 0 0 0 0)
   )
-  (no_connect (at 81.28 110.49))
+  (wire (pts (xy 73.66 110.49) (xy 81.28 110.49))
+    (stroke (width 0) (type default) (color 0 0 0 0))
+  )
   (wire (pts (xy 73.66 125.73) (xy 81.28 125.73))
     (stroke (width 0) (type default) (color 0 0 0 0))
@@
     (effects (font (size 1.27 1.27)) (justify left))
   )
+  (hierarchical_label "SOUT" (shape output) (at 73.66 110.49 180)
+    (effects (font (size 1.27 1.27)) (justify right))
+  )
   (hierarchical_label "8" (shape output) (at 119.38 110.49 0)

Commit message: Finish ledmatrix pcb reverse engineering.
Parts:
- removed C?: C, symbol Device:C
- removed U?: LC7932m, symbol ledmatrix:LC7932m
- added C7: (no value), symbol Device:C
- added U13: (no value), symbol ledmatrix:LC7932m
Connections:
- net 1: now also U13.25 (D1)
- net 10: now also U13.14 (D10)
- net 11: now also U13.12 (D11)
- net 12: now also U13.11 (D12)
- net 13: now also U13.10 (D13)
- net 14: now also U13.9 (D14)
- net 15: now also U13.7 (D15)
- net 16: now also U13.6 (D16)
- net 2: now also U13.24 (D2)
- net 3: now also U13.22 (D3)
- net 4: now also U13.21 (D4)
- net 5: now also U13.20 (D5)
- net 6: now also U13.19 (D6)
- net 7: now also U13.17 (D7)
- net 8: now also U13.16 (D8)
- net 9: now also U13.15 (D9)
- net CLOCK: now also U13.29 (CLOCK)
- net ENABLE: now also U13.2 (BEO)
- net GND: now also C7.2, U13.1 (VSS(L)), U13.13 (VSS(D)), U13.18 (VSS(D)), U13.23 (VSS(D)), U13.8 (VSS(D))
- net SIN: now also U13.5 (SOUT)
- net SOUT: now also U13.26 (SIN)
- net VCC: now also C7.1, U13.30 (VDD), U13.4 (L/R)
- net ~{LATCH}: now also U13.28 (~{LATCH})
- net ~{STROBE}: now also U13.3 (~{STROBE})
- no-connect marks 0 -> 1

Commit message: switch to desktop
Parts:
- C7, U13: value (none) -> ~
Changed lines of the file:
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@@
       (effects (font (size 1.27 1.27)) hide)
     )
-    (property "Value" "" (id 1) (at 135.89 138.43 0))
+    (property "Value" "~" (id 1) (at 135.89 138.43 0))
     (property "Footprint" "" (id 2) (at 135.89 134.62 0)
       (effects (font (size 1.27 1.27)) hide)
@@
       (effects (font (size 1.27 1.27)) (justify left))
     )
-    (property "Value" "" (id 1) (at 142.24 130.81 0)
+    (property "Value" "~" (id 1) (at 142.24 130.81 0)
       (effects (font (size 1.27 1.27)) (justify left))
     )
@@
       (effects (font (size 1.27 1.27)) hide)
     )
-    (property "Value" "" (id 1) (at 115.57 95.25 0))
+    (property "Value" "~" (id 1) (at 115.57 95.25 0))
     (property "Footprint" "" (id 2) (at 115.57 99.06 0)
       (effects (font (size 1.27 1.27)) hide)
@@
       (effects (font (size 1.27 1.27)) (justify left))
     )
-    (property "Value" "" (id 1) (at 135.89 60.96 0)
+    (property "Value" "~" (id 1) (at 135.89 60.96 0)
       (effects (font (size 1.27 1.27)) (justify left))
     )
@@
       (effects (font (size 1.27 1.27)) hide)
     )
-    (property "Value" "" (id 1) (at 135.89 72.39 0))
+    (property "Value" "~" (id 1) (at 135.89 72.39 0))
     (property "Footprint" "" (id 2) (at 135.89 76.2 0)
       (effects (font (size 1.27 1.27)) hide)
@@
       (effects (font (size 1.27 1.27)) hide)
     )
-    (property "Value" "" (id 1) (at 135.89 66.04 0))
+    (property "Value" "~" (id 1) (at 135.89 66.04 0))
     (property "Footprint" "" (id 2) (at 135.89 62.23 0)
       (effects (font (size 1.27 1.27)) hide)
@@
       (effects (font (size 1.27 1.27)) hide)
     )
-    (property "Value" "" (id 1) (at 135.89 50.8 0))
+    (property "Value" "~" (id 1) (at 135.89 50.8 0))
     (property "Footprint" "" (id 2) (at 135.89 54.61 0)
       (effects (font (size 1.27 1.27)) hide)
