File: ledmatrix/drivers.kicad_sch (KiCad schematic)
At the start: 94 parts, among them U1 74HC123, U2 74HC14, U3 74LS08, U4 74HC14

Commit message: switch to desktop
Parts:
- J1, J2, J3, J4: value (none) -> Conn_01x16
- J5: value (none) -> Conn_01x08
- JY1: value (none) -> Conn_01x24
- R10, R11, R12, R13, R14, R15, R16, R17, R18, R19, R20, R21, R22, R23, R24, R25, R26, R27, R28, R29, R3, R30, R31, R32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: value (none) -> R
- U5, U6: value (none) -> 74HC163
- U7, U8: value (none) -> 74HC4515
