File: ledmatrix/misc.kicad_sch (KiCad schematic)
At the start: 27 parts, among them U1 74HC123, U14 74HC74, U16 74LS32, U17 74HC14, U2 74HC14, U3 74LS08

Commit message: switch to desktop
Parts:
- C13: value (none) -> 1uF
- C9: value (none) -> 470uF
- D1: value (none) -> 1N4148
- J6: value (none) -> Conn_02x03_Top_Bottom
- J7: value (none) -> Conn_01x04
- R75: value (none) -> 10k
- R76: value (none) -> 120
- R77, R78: value (none) -> 4.7k
- R79, R80: value (none) -> 51k
- U15: value (none) -> S-8054ALR
- U18: value (none) -> SN75176AP
- U4: value (none) -> 74HC14
Changed lines of the file:
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@@
       (effects (font (size 1.27 1.27)) hide)
     )
-    (property "Value" "" (id 1) (at 201.93 53.34 0))
+    (property "Value" "GND" (id 1) (at 201.93 53.34 0))
     (property "Footprint" "" (id 2) (at 201.93 49.53 0)
       (effects (font (size 1.27 1.27)) hide)
@@
       (effects (font (size 1.27 1.27)) (justify left))
     )
-    (property "Value" "" (id 1) (at 118.11 40.64 0)
+    (property "Value" "1uF" (id 1) (at 118.11 40.64 0)
       (effects (font (size 1.27 1.27)) (justify left))
     )
@@
       (effects (font (size 1.27 1.27)) (justify left))
     )
-    (property "Value" "" (id 1) (at 189.23 36.83 90)
+    (property "Value" "120" (id 1) (at 189.23 36.83 90)
       (effects (font (size 1.27 1.27)) (justify left))
     )
@@
     (in_bom yes) (on_board yes)
     (property "Reference" "D1" (id 0) (at 114.3 22.86 0))
-    (property "Value" "" (id 1) (at 111.76 19.05 0))
+    (property "Value" "1N4148" (id 1) (at 111.76 19.05 0))
     (property "Footprint" "" (id 2) (at 111.76 21.59 0)
       (effects (font (size 1.27 1.27)) hide)
@@
       (effects (font (size 1.27 1.27)) (justify left))
     )
-    (property "Value" "" (id 1) (at 60.96 36.83 0)
+    (property "Value" "470uF" (id 1) (at 60.96 36.83 0)
       (effects (font (size 1.27 1.27)) (justify left))
     )
@@
       (effects (font (size 1.27 1.27)) hide)
     )
-    (property "Value" "" (id 1) (at 34.29 44.45 0))
+    (property "Value" "PWR_FLAG" (id 1) (at 34.29 44.45 0))
     (property "Footprint" "" (id 2) (at 34.29 40.64 0)
       (effects (font (size 1.27 1.27)) hide)
@@
       (effects (font (size 1.27 1.27)) (justify left))
     )
-    (property "Value" "" (id 1) (at 223.52 43.18 0)
+    (property "Value" "SN75176AP" (id 1) (at 223.52 43.18 0)
       (effects (font (size 1.27 1.27)) (justify left))
     )
@@
       (effects (font (size 1.27 1.27)) hide)
     )
-    (property "Value" "" (id 1) (at 212.09 20.32 0))
+    (property "Value" "VCC" (id 1) (at 212.09 20.32 0))
     (property "Footprint" "" (id 2) (at 212.09 24.13 0)
       (effects (font (size 1.27 1.27)) hide)
@@
       (effects (font (size 1.27 1.27)) hide)
     )
-    (property "Value" "" (id 1) (at 212.09 48.26 0))
+    (property "Value" "GND" (id 1) (at 212.09 48.26 0))
     (property "Footprint" "" (id 2) (at 212.09 44.45 0)
       (effects (font (size 1.27 1.27)) hide)
@@
       (effects (font (size 1.27 1.27)) hide)
     )
-    (property "Value" "" (id 1) (at 201.93 17.78 0))
+    (property "Value" "VCC" (id 1) (at 201.93 17.78 0))
     (property "Footprint" "" (id 2) (at 201.93 21.59 0)
       (effects (font (size 1.27 1.27)) hide)
@@
       (effects (font (size 1.27 1.27)) (justify right))
     )
-    (property "Value" "" (id 1) (at 107.95 38.1 0)
+    (property "Value" "S-8054ALR" (id 1) (at 107.95 38.1 0)
       (effects (font (size 1.27 1.27)) (justify right))
     )
@@
       (effects (font (size 1.27 1.27)) hide)
     )
-    (property "Value" "" (id 1) (at 96.52 20.32 0))
+    (property "Value" "VCC" (id 1) (at 96.52 20.32 0))
     (property "Footprint" "" (id 2) (at 96.52 24.13 0)
       (effects (font (size 1.27 1.27)) hide)
@@
     (in_bom yes) (on_board yes)
     (property "Reference" "R78" (id 0) (at 194.31 36.83 90))
-    (property "Value" "" (id 1) (at 195.58 39.37 90))
+    (property "Value" "4.7k" (id 1) (at 195.58 39.37 90))
     (property "Footprint" "" (id 2) (at 195.58 41.148 90)
       (effects (font (size 1.27 1.27)) hide)
@@
       (effects (font (size 1.27 1.27)) hide)
     )
-    (property "Value" "" (id 1) (at 34.29 24.13 0))
+    (property "Value" "PWR_FLAG" (id 1) (at 34.29 24.13 0))
     (property "Footprint" "" (id 2) (at 34.29 27.94 0)
       (effects (font (size 1.27 1.27)) hide)
@@
       (effects (font (size 1.27 1.27)) (justify left))
     )
-    (property "Value" "" (id 1) (at 201.93 46.99 90)
+    (property "Value" "51k" (id 1) (at 201.93 46.99 90)
       (effects (font (size 1.27 1.27)) (justify left))
     )
@@
       (effects (font (size 1.27 1.27)) (justify left))
     )
-    (property "Value" "" (id 1) (at 201.93 26.67 90)
+    (property "Value" "51k" (id 1) (at 201.93 26.67 90)
       (effects (font (size 1.27 1.27)) (justify left))
     )
@@
       (effects (font (size 1.27 1.27)) hide)
     )
-    (property "Value" "" (id 1) (at 226.06 33.02 0))
+    (property "Value" "GND" (id 1) (at 226.06 33.02 0))
     (property "Footprint" "" (id 2) (at 226.06 29.21 0)
       (effects (font (size 1.27 1.27)) hide)
@@
     (in_bom yes) (on_board yes)
     (property "Reference" "J7" (id 0) (at 177.8 29.21 0))
-    (property "Value" "" (id 1) (at 177.8 41.91 0))
+    (property "Value" "Conn_01x04" (id 1) (at 177.8 41.91 0))
     (property "Footprint" "" (id 2) (at 177.8 34.29 0)
       (effects (font (size 1.27 1.27)) hide)
@@
       (effects (font (size 1.27 1.27)) hide)
     )
-    (property "Value" "" (id 1) (at 118.11 45.72 0))
+    (property "Value" "GND" (id 1) (at 118.11 45.72 0))
     (property "Footprint" "" (id 2) (at 118.11 41.91 0)
       (effects (font (size 1.27 1.27)) hide)
@@
     (in_bom yes) (on_board yes)
     (property "Reference" "R77" (id 0) (at 194.31 29.21 90))
-    (property "Value" "" (id 1) (at 195.58 31.75 90))
+    (property "Value" "4.7k" (id 1) (at 195.58 31.75 90))
     (property "Footprint" "" (id 2) (at 195.58 33.528 90)
       (effects (font (size 1.27 1.27)) hide)
@@
     (in_bom yes) (on_board yes)
     (property "Reference" "U4" (id 0) (at 132.08 40.64 0))
-    (property "Value" "" (id 1) (at 132.08 49.53 0))
+    (property "Value" "74HC14" (id 1) (at 132.08 49.53 0))
     (property "Footprint" "" (id 2) (at 132.08 44.45 0)
       (effects (font (size 1.27 1.27)) hide)
@@
       (effects (font (size 1.27 1.27)) hide)
     )
-    (property "Value" "" (id 1) (at 96.52 43.18 0))
+    (property "Value" "GND" (id 1) (at 96.52 43.18 0))
     (property "Footprint" "" (id 2) (at 96.52 39.37 0)
       (effects (font (size 1.27 1.27)) hide)
@@
     (in_bom yes) (on_board yes)
     (property "Reference" "U4" (id 0) (at 132.08 27.94 0))
-    (property "Value" "" (id 1) (at 132.08 36.83 0))
+    (property "Value" "74HC14" (id 1) (at 132.08 36.83 0))
     (property "Footprint" "" (id 2) (at 132.08 31.75 0)
       (effects (font (size 1.27 1.27)) hide)
@@
       (effects (font (size 1.27 1.27)) hide)
     )
-    (property "Value" "" (id 1) (at 64.77 44.45 0))
+    (property "Value" "GND" (id 1) (at 64.77 44.45 0))
     (property "Footprint" "" (id 2) (at 64.77 40.64 0)
       (effects (font (size 1.27 1.27)) hide)
@@
       (effects (font (size 1.27 1.27)) hide)
     )
-    (property "Value" "" (id 1) (at 64.77 24.13 0))
+    (property "Value" "VCC" (id 1) (at 64.77 24.13 0))
     (property "Footprint" "" (id 2) (at 64.77 27.94 0)
       (effects (font (size 1.27 1.27)) hide)
@@
     (in_bom yes) (on_board yes)
     (property "Reference" "J6" (id 0) (at 36.83 34.29 0))
-    (property "Value" "" (id 1) (at 46.99 38.1 90))
+    (property "Value" "Conn_02x03_Top_Bottom" (id 1) (at 46.99 38.1 90))
     (property "Footprint" "" (id 2) (at 31.75 33.02 0)
       (effects (font (size 1.27 1.27)) hide)
@@
     (in_bom yes) (on_board yes)
     (property "Reference" "R75" (id 0) (at 113.03 29.21 90))
-    (property "Value" "" (id 1) (at 111.76 31.75 90))
+    (property "Value" "10k" (id 1) (at 111.76 31.75 90))
     (property "Footprint" "" (id 2) (at 111.76 33.528 90)
       (effects (font (size 1.27 1.27)) hide)
