File: ledmatrix/lcdcontroller.kicad_sch (KiCad schematic)
At the start: 9 parts, among them U3 74LS08, U4 74HC14

Commit message: switch to desktop
Parts:
- U14: value (none) -> 74HC74
- U19: value (none) -> SED1351F
- U20: value (none) -> 74HC166
- U21: value (none) -> LC36128ML
Changed lines of the file:
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@@
       (effects (font (size 1.27 1.27)) hide)
     )
-    (property "Value" "" (id 1) (at 92.71 22.86 0))
+    (property "Value" "VCC" (id 1) (at 92.71 22.86 0))
     (property "Footprint" "" (id 2) (at 92.71 26.67 0)
       (effects (font (size 1.27 1.27)) hide)
@@
       (effects (font (size 1.27 1.27)) hide)
     )
-    (property "Value" "" (id 1) (at 44.45 62.23 0))
+    (property "Value" "GND" (id 1) (at 44.45 62.23 0))
     (property "Footprint" "" (id 2) (at 44.45 58.42 0)
       (effects (font (size 1.27 1.27)) hide)
@@
       (effects (font (size 1.27 1.27)) hide)
     )
-    (property "Value" "" (id 1) (at 36.83 157.48 0))
+    (property "Value" "VCC" (id 1) (at 36.83 157.48 0))
     (property "Footprint" "" (id 2) (at 36.83 161.29 0)
       (effects (font (size 1.27 1.27)) hide)
@@
       (effects (font (size 1.27 1.27)) hide)
     )
-    (property "Value" "" (id 1) (at 29.21 172.72 0))
+    (property "Value" "VCC" (id 1) (at 29.21 172.72 0))
     (property "Footprint" "" (id 2) (at 29.21 176.53 0)
       (effects (font (size 1.27 1.27)) hide)
@@
       (effects (font (size 1.27 1.27)) hide)
     )
-    (property "Value" "" (id 1) (at 44.45 134.62 0))
+    (property "Value" "VCC" (id 1) (at 44.45 134.62 0))
     (property "Footprint" "" (id 2) (at 44.45 138.43 0)
       (effects (font (size 1.27 1.27)) hide)
@@
     (in_bom yes) (on_board yes)
     (property "Reference" "U20" (id 0) (at 118.11 152.4 0))
-    (property "Value" "" (id 1) (at 121.92 185.42 0))
+    (property "Value" "74HC166" (id 1) (at 121.92 185.42 0))
     (property "Footprint" "" (id 2) (at 128.27 181.61 0)
       (effects (font (size 1.27 1.27)) hide)
@@
     (in_bom yes) (on_board yes)
     (property "Reference" "U19" (id 0) (at 87.63 22.86 0))
-    (property "Value" "" (id 1) (at 85.09 177.8 0))
+    (property "Value" "SED1351F" (id 1) (at 85.09 177.8 0))
     (property "Footprint" "" (id 2) (at 81.28 46.99 0)
       (effects (font (size 1.27 1.27)) hide)
@@
       (effects (font (size 1.27 1.27)) hide)
     )
-    (property "Value" "" (id 1) (at 49.53 22.86 0))
+    (property "Value" "VCC" (id 1) (at 49.53 22.86 0))
     (property "Footprint" "" (id 2) (at 49.53 26.67 0)
       (effects (font (size 1.27 1.27)) hide)
@@
       (effects (font (size 1.27 1.27)) hide)
     )
-    (property "Value" "" (id 1) (at 148.59 33.02 0))
+    (property "Value" "VCC" (id 1) (at 148.59 33.02 0))
     (property "Footprint" "" (id 2) (at 148.59 36.83 0)
       (effects (font (size 1.27 1.27)) hide)
@@
       (effects (font (size 1.27 1.27)) hide)
     )
-    (property "Value" "" (id 1) (at 147.32 185.42 0))
+    (property "Value" "GND" (id 1) (at 147.32 185.42 0))
     (property "Footprint" "" (id 2) (at 147.32 181.61 0)
       (effects (font (size 1.27 1.27)) hide)
@@
       (effects (font (size 1.27 1.27)) hide)
     )
-    (property "Value" "" (id 1) (at 111.76 152.4 0))
+    (property "Value" "VCC" (id 1) (at 111.76 152.4 0))
     (property "Footprint" "" (id 2) (at 111.76 156.21 0)
       (effects (font (size 1.27 1.27)) hide)
@@
       (effects (font (size 1.27 1.27)) hide)
     )
-    (property "Value" "" (id 1) (at 149.86 152.4 0))
+    (property "Value" "VCC" (id 1) (at 149.86 152.4 0))
     (property "Footprint" "" (id 2) (at 149.86 156.21 0)
       (effects (font (size 1.27 1.27)) hide)
@@
       (effects (font (size 1.27 1.27)) hide)
     )
-    (property "Value" "" (id 1) (at 97.79 114.3 0))
+    (property "Value" "VCC" (id 1) (at 97.79 114.3 0))
     (property "Footprint" "" (id 2) (at 97.79 118.11 0)
       (effects (font (size 1.27 1.27)) hide)
@@
     (in_bom yes) (on_board yes)
     (property "Reference" "U21" (id 0) (at 144.78 33.02 0))
-    (property "Value" "" (id 1) (at 140.97 101.6 0))
+    (property "Value" "LC36128ML" (id 1) (at 140.97 101.6 0))
     (property "Footprint" "" (id 2) (at 133.35 67.31 0)
       (effects (font (size 1.27 1.27)) hide)
@@
       (effects (font (size 1.27 1.27)) hide)
     )
-    (property "Value" "" (id 1) (at 148.59 76.2 0))
+    (property "Value" "GND" (id 1) (at 148.59 76.2 0))
     (property "Footprint" "" (id 2) (at 148.59 72.39 0)
       (effects (font (size 1.27 1.27)) hide)
@@
       (effects (font (size 1.27 1.27)) hide)
     )
-    (property "Value" "" (id 1) (at 49.53 177.8 0))
+    (property "Value" "GND" (id 1) (at 49.53 177.8 0))
     (property "Footprint" "" (id 2) (at 49.53 173.99 0)
       (effects (font (size 1.27 1.27)) hide)
@@
       (effects (font (size 1.27 1.27)) hide)
     )
-    (property "Value" "" (id 1) (at 151.13 172.72 0))
+    (property "Value" "VCC" (id 1) (at 151.13 172.72 0))
     (property "Footprint" "" (id 2) (at 151.13 176.53 0)
       (effects (font (size 1.27 1.27)) hide)
@@
       (effects (font (size 1.27 1.27)) hide)
     )
-    (property "Value" "" (id 1) (at 92.71 177.8 0))
+    (property "Value" "GND" (id 1) (at 92.71 177.8 0))
     (property "Footprint" "" (id 2) (at 92.71 173.99 0)
       (effects (font (size 1.27 1.27)) hide)
@@
     (in_bom yes) (on_board yes)
     (property "Reference" "U14" (id 0) (at 39.37 162.56 0))
-    (property "Value" "" (id 1) (at 40.64 175.26 0))
+    (property "Value" "74HC74" (id 1) (at 40.64 175.26 0))
     (property "Footprint" "" (id 2) (at 36.83 168.91 0)
       (effects (font (size 1.27 1.27)) hide)
@@
       (effects (font (size 1.27 1.27)) hide)
     )
-    (property "Value" "" (id 1) (at 44.45 64.77 0))
+    (property "Value" "VCC" (id 1) (at 44.45 64.77 0))
     (property "Footprint" "" (id 2) (at 44.45 68.58 0)
       (effects (font (size 1.27 1.27)) hide)
