File: ledmatrix/ledmatrix.kicad_sch (KiCad schematic)
At the start: 0 parts

Commit message: Finish ledmatrix pcb reverse engineering.
Other:
- sheet comms renamed misc
- removed sheet scanlines
- added sheet lcdcontroller (lcdcontroller.kicad_sch)
- added sheet memory (memory.kicad_sch)
- added sheet mpu (mpu.kicad_sch)
- sheet misc: file comms.kicad_sch -> misc.kicad_sch
- sheet misc ports: added RESET, RX, ~{RESET}; removed none

Commit message: switch to desktop
Other:
- sheet memory ports: added PIN16(~{IORQ}), PIN33(~{M1}); removed PIN16(~{CONCS}), PIN33(CONCS)
