File: pulse_shorter/pulse_shorter.kicad_sch (KiCad schematic)
At the start: 5 parts, among them J1 Conn_01x03, J2 Conn_01x03, U1 4093

Commit message: Add comment about RC values
Other:
- note added: "Pick R and C so that RC ~= 200ns. i.e. R = 10k C = 22pF"
Changed lines of the file:
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@@
     (stroke (width 0) (type default) (color 0 0 0 0))
+  )
+  (text "Pick R and C so that RC ~= 200ns. i.e.\nR = 10k\nC = 22pF"
+    (at 130.81 54.61 0)
+    (effects (font (size 1.27 1.27)) (justify left bottom))
   )
   (symbol (lib_id "Connector_Generic:Conn_01x03") (at 198.12 36.83 0) (mirror x) (unit 1)
