File: ledpcb/ledpcb-ws2813/ledpcb-ws2813.kicad_sch (KiCad schematic)
At the start: 37 parts, among them J1 JST_XA_B04B, J2 JST_XA_B03B, J3 JST_XA_B03B

Commit message: Merge some changes between desktop and laptop manually...
Other:
- note added: "If using ws2813b's populate R1-6,8,10 and C1-2,4-9. If using ws2813b-v5's then pin 1 changes from VCC to BOUT, which is internally connected to DIN (experimentally confirmed). In this case, do not populate the above mentioned resistors and capacitors."
Changed lines of the file:
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@@
     (stroke (width 0) (type default) (color 0 0 0 0))
+  )
+  (text "If using ws2813b's populate R1-6,8,10 and C1-2,4-9.\nIf using ws2813b-v5's then pin 1 changes from VCC to BOUT,\nwhich is internally connected to DIN (experimentally confirmed).\nIn this case, do not populate the above mentioned resistors and capacitors."
+    (at 40.64 115.57 0)
+    (effects (font (size 1.27 1.27)) (justify left bottom))
   )
   (label "DATA OUT" (at 228.6 80.01 0)

Commit message: replace C110526 by C2844869
Parts:
- ZD1: LCSC C110526 -> C2844869
Changed lines of the file:
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@@
       (effects (font (size 1.27 1.27)) hide)
     )
-    (property "LCSC" "C110526" (id 5) (at 140.97 114.3 0)
+    (property "LCSC" "C2844869" (id 5) (at 140.97 114.3 0)
       (effects (font (size 1.27 1.27)) hide)
     )

Commit message: move zd1 from 1SMA4734 to 1SMA4734A.
Parts:
- ZD1: LCSC C2844869 -> C5128847
Changed lines of the file:
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@@
       (effects (font (size 1.27 1.27)) hide)
     )
-    (property "LCSC" "C2844869" (id 5) (at 140.97 114.3 0)
+    (property "LCSC" "C5128847" (id 5) (at 140.97 114.3 0)
       (effects (font (size 1.27 1.27)) hide)
     )
